File: dc-dc_12-5.kicad_sch (KiCad schematic)
At the start: 7 parts, among them U601 TPS562202

Commit message: Found IC for ORing function. Added all LCSC refs. Found proper header stackup.
Signed-off-by: Jean Alinei <jean.alinei@owntech.org>
Parts:
- C601: LCSC (none) -> C440198; Reserved1 3c8c36ffa6a0eb88db22fa786b0d8984706c66e773e3ba -> (none)
- C602: footprint Capacitor_SMD:C_0805_2012Metric -> Capacitor_SMD:C_0603_1608Metric; LCSC (none) -> C14663; Reserved1 19d8e62435aae811d30466f8cc008899f37785f68fd5 -> (none)
- C603: LCSC (none) -> C96123; Reserved1 31dd9bc8149be90ead65bb5faf8babf00b42c01fb99f -> (none)
- L601: LCSC (none) -> C3002596; Reserved1 4b5e7131c4b8cb9d5c96e3b4c03b6959f47985d47fcfaf65 -> (none)
- R601: footprint Footprints:R_0805_2012Metric -> Resistor_SMD:R_0603_1608Metric; LCSC (none) -> C23206; Reserved1 40c9798757babe36703e44e551b8c4e5a4b8adf8358a -> (none)
- R602: footprint Footprints:R_0805_2012Metric -> Resistor_SMD:R_0603_1608Metric; LCSC (none) -> C25804; Reserved1 9643e47a19e72e78ce6b1a1e2bf5602d194d9ae39a95 -> (none)
- U601: LCSC (none) -> C2877547; Reserved1 bdd6eb54c347894819d6b847551483c266f534e32b90e02b -> (none)

Commit message: Added datasheets & updated components descriptions & values
Signed-off-by: Jean Alinei <jean.alinei@owntech.org>
Parts:
- U601: value TPS562202 -> TPS562202DRLR
Changed lines of the file:
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@@
 			)
 		)
-		(property "Description" "Resistor, small symbol"
+		(property "Description" "10kΩ ±1% 100mW 0603 Thick Film Resistor"
 			(at 114.3 97.79 0)
 			(hide yes)
@@
 			)
 		)
-		(property "Description" "Unpolarized capacitor"
+		(property "Description" "47uF ±20% 10V Ceramic Capacitor X5R 1206"
 			(at 124.46 93.98 0)
 			(hide yes)
@@
 			)
 		)
-		(property "Value" "TPS562202"
+		(property "Value" "TPS562202DRLR"
 			(at 78.74 80.01 0)
 			(show_name no)
@@
 			)
 		)
-		(property "Description" "2A Synchronous Step-Down Voltage Regulator 580kHz, adjustable output voltage, 4.5-17V Input Voltage, 0.804V-7V Output Voltage, SOT-563"
+		(property "Description" "Buck Switching Regulator IC Adjustable 0.804V~7V 1 Output 2A SOT-6(3x5)"
 			(at 78.74 87.63 0)
 			(hide yes)
@@
 			)
 		)
-		(property "Description" "Unpolarized capacitor"
+		(property "Description" "10uF ±10% 50V Ceramic Capacitor X5R 0805"
 			(at 53.34 93.98 0)
 			(hide yes)
@@
 			)
 		)
-		(property "Description" "Inductor"
+		(property "Description" "2.2A 4.7uH ±20% 126mΩ 3A Molded inductor SMD,4.6x4.1mm Fixed Inductors RoHS"
 			(at 107.95 85.09 0)
 			(hide yes)
@@
 			)
 		)
-		(property "Description" "Unpolarized capacitor, small symbol"
+		(property "Description" "100nF ±10% 50V Ceramic Capacitor X7R 0603"
 			(at 93.98 87.63 0)
 			(hide yes)
@@
 			)
 		)
-		(property "Description" "Resistor, small symbol"
+		(property "Description" "56kΩ ±1% 100mW 0603 Thick Film Resistor"
 			(at 114.3 90.17 0)
 			(hide yes)
