File: Feeder.kicad_sch (KiCad schematic)
At the start: 48 parts, among them J101 PZ254V-22-06-A60-1500, J102 PZ254V-21-03-A60-1500, U101 24C02S(XBLW), U102 MX5050S3028A2

Commit message: Added rotation offsets.
Signed-off-by: Jean Alinei <jean.alinei@owntech.org>
Parts:
- C107, C108, C109, C110, C111, C112, C113, C114, C115, C116, C117, C118: Rotation Offset (none) -> 180
- J101, J102: Rotation Offset (none) -> 90
Other:
- moved on the sheet: J101
