File: dc-dc_12-6.kicad_sch (KiCad schematic)
At the start: 7 parts, among them U601 TPS562202

Commit message: First layout complete - DRC not clear yet.
Signed-off-by: Jean Alinei <jean.alinei@owntech.org>
Parts:
- renumbered C601 to C701, C602 to C702, C603 to C703, L601 to L701, R601 to R701, R602 to R702, U601 to U701
Changed lines of the file:
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@@
 		(polyline
 			(pts
-				(xy 33.02 64.77) (xy 33.02 116.84) (xy 154.94 116.84) (xy 154.94 64.77)
+				(xy 33.02 66.04) (xy 33.02 116.84) (xy 153.67 116.84) (xy 153.67 66.04)
 			)
 			(stroke
 				(width 0)
 				(type solid)
-				(color 0 194 0 1)
+				(color 0 0 194 1)
 			)
 			(fill
 				(type color)
-				(color 0 194 0 0.1019607843)
+				(color 0 0 194 0.1019607843)
 			)
 		)
@@
 			(justify left bottom)
 		)
-		(property "Netclass" "DGND"
+		(property "Netclass" "PGND"
 			(at 37.4396 114.3 0)
 			(show_name no)
@@
 		(in_pos_files yes)
 		(dnp no)
-		(property "Reference" "R602"
+		(property "Reference" "R702"
 			(at 116.84 96.5199 0)
 			(show_name no)
@@
 		(instances
 			(project "Feeder"
-				(path "/8d0c1d66-35ef-4a53-a28f-436a11b54f42/08fa4b66-394b-4012-88ba-dcadeef448ea"
-					(reference "R602")
+				(path "/8d0c1d66-35ef-4a53-a28f-436a11b54f42/80c75c33-7ca5-47fa-98cc-678becbdce40"
+					(reference "R702")
 					(unit 1)
 				)
@@
 		(in_pos_files yes)
 		(dnp no)
-		(property "Reference" "C603"
+		(property "Reference" "C703"
 			(at 128.27 92.7099 0)
 			(show_name no)
@@
 		(instances
 			(project "Feeder"
-				(path "/8d0c1d66-35ef-4a53-a28f-436a11b54f42/08fa4b66-394b-4012-88ba-dcadeef448ea"
-					(reference "C603")
+				(path "/8d0c1d66-35ef-4a53-a28f-436a11b54f42/80c75c33-7ca5-47fa-98cc-678becbdce40"
+					(reference "C703")
 					(unit 1)
 				)
@@
 		(dnp no)
 		(fields_autoplaced yes)
-		(property "Reference" "U601"
+		(property "Reference" "U701"
 			(at 78.74 77.47 0)
 			(show_name no)
@@
 		(instances
 			(project "Feeder"
-				(path "/8d0c1d66-35ef-4a53-a28f-436a11b54f42/08fa4b66-394b-4012-88ba-dcadeef448ea"
-					(reference "U601")
+				(path "/8d0c1d66-35ef-4a53-a28f-436a11b54f42/80c75c33-7ca5-47fa-98cc-678becbdce40"
+					(reference "U701")
 					(unit 1)
 				)
@@
 		(dnp no)
 		(fields_autoplaced yes)
-		(property "Reference" "C601"
+		(property "Reference" "C701"
 			(at 57.15 92.7099 0)
 			(show_name no)
@@
 		(instances
 			(project "Feeder"
-				(path "/8d0c1d66-35ef-4a53-a28f-436a11b54f42/08fa4b66-394b-4012-88ba-dcadeef448ea"
-					(reference "C601")
+				(path "/8d0c1d66-35ef-4a53-a28f-436a11b54f42/80c75c33-7ca5-47fa-98cc-678becbdce40"
+					(reference "C701")
 					(unit 1)
 				)
@@
 		(in_pos_files yes)
 		(dnp no)
-		(property "Reference" "L601"
+		(property "Reference" "L701"
 			(at 107.95 80.01 90)
 			(show_name no)
@@
 		(instances
 			(project "Feeder"
-				(path "/8d0c1d66-35ef-4a53-a28f-436a11b54f42/08fa4b66-394b-4012-88ba-dcadeef448ea"
-					(reference "L601")
+				(path "/8d0c1d66-35ef-4a53-a28f-436a11b54f42/80c75c33-7ca5-47fa-98cc-678becbdce40"
+					(reference "L701")
 					(unit 1)
 				)
@@
 		(in_pos_files yes)
 		(dnp no)
-		(property "Reference" "C602"
+		(property "Reference" "C702"
 			(at 98.044 89.408 90)
 			(show_name no)
@@
 		(instances
 			(project "Feeder"
-				(path "/8d0c1d66-35ef-4a53-a28f-436a11b54f42/08fa4b66-394b-4012-88ba-dcadeef448ea"
-					(reference "C602")
+				(path "/8d0c1d66-35ef-4a53-a28f-436a11b54f42/80c75c33-7ca5-47fa-98cc-678becbdce40"
+					(reference "C702")
 					(unit 1)
 				)
@@
 		(in_pos_files yes)
 		(dnp no)
-		(property "Reference" "R601"
+		(property "Reference" "R701"
 			(at 116.84 88.8999 0)
 			(show_name no)
@@
 		(instances
 			(project "Feeder"
-				(path "/8d0c1d66-35ef-4a53-a28f-436a11b54f42/08fa4b66-394b-4012-88ba-dcadeef448ea"
-					(reference "R601")
+				(path "/8d0c1d66-35ef-4a53-a28f-436a11b54f42/80c75c33-7ca5-47fa-98cc-678becbdce40"
+					(reference "R701")
 					(unit 1)
 				)
@@
 		(in_pos_files yes)
 		(dnp no)
-		(property "Reference" "#FLG0601"
+		(property "Reference" "#FLG0701"
 			(at 132.08 80.645 0)
 			(hide yes)
@@
 		(instances
 			(project "Feeder"
-				(path "/8d0c1d66-35ef-4a53-a28f-436a11b54f42/08fa4b66-394b-4012-88ba-dcadeef448ea"
-					(reference "#FLG0601")
+				(path "/8d0c1d66-35ef-4a53-a28f-436a11b54f42/80c75c33-7ca5-47fa-98cc-678becbdce40"
+					(reference "#FLG0701")
 					(unit 1)
 				)

Commit message: Found IC for ORing function. Added all LCSC refs. Found proper header stackup.
Signed-off-by: Jean Alinei <jean.alinei@owntech.org>
Parts:
- C701: LCSC (none) -> C440198; Reserved1 3c8c36ffa6a0eb88db22fa786b0d8984706c66e773e3ba -> (none)
- C702: footprint Capacitor_SMD:C_0805_2012Metric -> Capacitor_SMD:C_0603_1608Metric; LCSC (none) -> C14663; Reserved1 19d8e62435aae811d30466f8cc008899f37785f68fd5 -> (none)
- C703: LCSC (none) -> C96123; Reserved1 31dd9bc8149be90ead65bb5faf8babf00b42c01fb99f -> (none)
- L701: LCSC (none) -> C3002596; Reserved1 4b5e7131c4b8cb9d5c96e3b4c03b6959f47985d47fcfaf65 -> (none)
- R701: footprint Footprints:R_0805_2012Metric -> Resistor_SMD:R_0603_1608Metric; LCSC (none) -> C23206; Reserved1 40c9798757babe36703e44e551b8c4e5a4b8adf8358a -> (none)
- R702: footprint Footprints:R_0805_2012Metric -> Resistor_SMD:R_0603_1608Metric; LCSC (none) -> C25804; Reserved1 9643e47a19e72e78ce6b1a1e2bf5602d194d9ae39a95 -> (none)
- U701: LCSC (none) -> C2877547; Reserved1 bdd6eb54c347894819d6b847551483c266f534e32b90e02b -> (none)

Commit message: Added datasheets & updated components descriptions & values
Signed-off-by: Jean Alinei <jean.alinei@owntech.org>
Parts:
- U701: value TPS562202 -> TPS562202DRLR
Changed lines of the file:
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@@
 			)
 		)
-		(property "Description" "Resistor, small symbol"
+		(property "Description" "10kΩ ±1% 100mW 0603 Thick Film Resistor"
 			(at 114.3 97.79 0)
 			(hide yes)
@@
 			)
 		)
-		(property "Description" "Unpolarized capacitor"
+		(property "Description" "47uF ±20% 10V Ceramic Capacitor X5R 1206"
 			(at 124.46 93.98 0)
 			(hide yes)
@@
 			)
 		)
-		(property "Value" "TPS562202"
+		(property "Value" "TPS562202DRLR"
 			(at 78.74 80.01 0)
 			(show_name no)
@@
 			)
 		)
-		(property "Description" "2A Synchronous Step-Down Voltage Regulator 580kHz, adjustable output voltage, 4.5-17V Input Voltage, 0.804V-7V Output Voltage, SOT-563"
+		(property "Description" "Buck Switching Regulator IC Adjustable 0.804V~7V 1 Output 2A SOT-6(3x5)"
 			(at 78.74 87.63 0)
 			(hide yes)
@@
 			)
 		)
-		(property "Description" "Unpolarized capacitor"
+		(property "Description" "10uF ±10% 50V Ceramic Capacitor X5R 0805"
 			(at 53.34 93.98 0)
 			(hide yes)
@@
 			)
 		)
-		(property "Description" "Inductor"
+		(property "Description" "2.2A 4.7uH ±20% 126mΩ 3A Molded inductor SMD,4.6x4.1mm Fixed Inductors RoHS"
 			(at 107.95 85.09 0)
 			(hide yes)
@@
 			)
 		)
-		(property "Description" "Unpolarized capacitor, small symbol"
+		(property "Description" "100nF ±10% 50V Ceramic Capacitor X7R 0603"
 			(at 93.98 87.63 0)
 			(hide yes)
@@
 			)
 		)
-		(property "Description" "Resistor, small symbol"
+		(property "Description" "56kΩ ±1% 100mW 0603 Thick Film Resistor"
 			(at 114.3 90.17 0)
 			(hide yes)
