File: dc-dc_isolated.kicad_sch (KiCad schematic)
At the start: 11 parts, among them U801 CMP6793RE

Commit message: First layout complete - DRC not clear yet.
Signed-off-by: Jean Alinei <jean.alinei@owntech.org>
Other:
- moved on the sheet: C801, C802, C803, C804, D801, D802, L801, R801, R802, TR801, U801

Commit message: Found IC for ORing function. Added all LCSC refs. Found proper header stackup.
Signed-off-by: Jean Alinei <jean.alinei@owntech.org>
Parts:
- TR801: LCSC (none) -> C37648313

Commit message: Added datasheets & updated components descriptions & values
Signed-off-by: Jean Alinei <jean.alinei@owntech.org>
Parts:
- D801, D802: value PMEG4010 -> PMEG4010ESBYL
Changed lines of the file:
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@@
 			)
 		)
-		(property "Description" "Unpolarized capacitor"
+		(property "Description" "100nF ±10% 50V Ceramic Capacitor X7R 0603"
 			(at 60.96 39.37 0)
 			(hide yes)
@@
 			)
 		)
-		(property "Description" "Unpolarized capacitor"
+		(property "Description" "10uF ±10% 50V Ceramic Capacitor X5R 0805"
 			(at 46.99 39.37 0)
 			(hide yes)
@@
 			)
 		)
-		(property "Value" "PMEG4010"
+		(property "Value" "PMEG4010ESBYL"
 			(at 155.448 44.704 0)
 			(show_name no)
@@
 			)
 		)
-		(property "Description" "Schottky diode, small symbol"
+		(property "Description" "Diode 40V 1A Surface Mount DSN1006-2"
 			(at 151.13 46.99 0)
 			(hide yes)
@@
 			)
 		)
-		(property "Description" "Unpolarized capacitor"
+		(property "Description" "10uF ±10% 50V Ceramic Capacitor X5R 0805"
 			(at 173.99 34.29 0)
 			(hide yes)
@@
 			)
 		)
-		(property "Value" "PMEG4010"
+		(property "Value" "PMEG4010ESBYL"
 			(at 145.542 26.67 0)
 			(show_name no)
@@
 			)
 		)
-		(property "Description" "Schottky diode, small symbol"
+		(property "Description" "Diode 40V 1A Surface Mount DSN1006-2"
 			(at 151.13 29.21 0)
 			(hide yes)
@@
 			)
 		)
-		(property "Description" "Isolated power transformer driver"
+		(property "Description" "ESOP-8 Power Management - Specialized RoHS"
 			(at 109.22 38.1 0)
 			(hide yes)
@@
 			)
 		)
-		(property "Description" "Unpolarized capacitor"
+		(property "Description" "10uF ±10% 50V Ceramic Capacitor X5R 0805"
 			(at 33.02 39.37 0)
 			(hide yes)
@@
 			)
 		)
-		(property "Description" "Inductor"
+		(property "Description" "350mA 10uH ±20% 150mA 470mΩ Multilayer inductor 0805 Fixed Inductors RoHS"
 			(at 40.64 26.67 0)
 			(hide yes)
