File: dc-dc_isolated_disabling.kicad_sch (KiCad schematic)
At the start: 11 parts, among them U801 CMP6793RE

Commit message: v2 wip
Parts:
- removed C801, C802, C804: 10uF, Capacitor_SMD:C_0805_2012Metric, symbol Device:C
- removed C803: 100nF, Capacitor_SMD:C_0603_1608Metric, symbol Device:C
- removed D801, D802: PMEG4010, Diode_SMD:D_SOD-882, symbol Device:D_Schottky_Small
- removed L801: 10uH, Inductor_SMD:L_0805_2012Metric, symbol Device:L
- removed R801: R_Small, Resistor_SMD:R_0603_1608Metric, symbol Device:R_Small
- removed R802: 4.7k, Resistor_SMD:R_0603_1608Metric, symbol Device:R_Small
- removed TR801: CMT88F0U, feeder:CMT88F0U, symbol feeder:CMT88F0U
- removed U801: CMP6793RE, Package_SO:SOIC-8-1EP_3.9x4.9mm_P1.27mm_EP2.41x3.3mm_ThermalVias, symbol feeder:CMP6793RE
- added C201, C202, C204: 10uF, Capacitor_SMD:C_0805_2012Metric, symbol Device:C
- added C203: 100nF, Capacitor_SMD:C_0603_1608Metric, symbol Device:C
- added D201, D202: PMEG4010, Diode_SMD:D_SOD-882, symbol Device:D_Schottky_Small
- added L201: 10uH, Inductor_SMD:L_0805_2012Metric, symbol Device:L
- added Q201: 2N7002, Package_TO_SOT_SMD:SOT-23, symbol Transistor_FET:2N7002
- added R202: 100k, Resistor_SMD:R_0603_1608Metric, symbol Device:R_Small
- added R203: R_Small, Resistor_SMD:R_0603_1608Metric, symbol Device:R_Small
- added R204: 4.7k, Resistor_SMD:R_0603_1608Metric, symbol Device:R_Small
- added TR201: CMT88F0U, feeder:CMT88F0U, symbol feeder:CMT88F0U
- added U201: CMP6793RE, Package_SO:SOIC-8-1EP_3.9x4.9mm_P1.27mm_EP2.41x3.3mm_ThermalVias, symbol feeder:CMP6793RE
Connections:
- net GND: now also C201.2, C202.2, C203.2, Q201.2 (S), R203.2, U201.2 (GND), U201.9 (GND)
- net OUT_GND: now also C204.2, R204.2, TR201.6, TR201.7
- net VIN: now also C201.1, L201.1
- net VOUT: now also C204.1, D201.1 (K), D202.1 (K), R204.1
- new net: D202.2 (A), TR201.5
- new net: Q201.3 (D), R202.2, U201.4 (EN)
- new net: R203.1, U201.1 (CLK)
- new net: D201.2 (A), TR201.8
- new net: C202.1, C203.1, L201.2, R202.1, U201.3 (VCC)
- new net: TR201.1, U201.5 (VD1)
- new net: TR201.4, U201.8 (VD2)
- new net ~{EN}: Q201.1 (G)

Commit message: First layout complete - DRC not clear yet.
Signed-off-by: Jean Alinei <jean.alinei@owntech.org>
Other:
- moved on the sheet: C201, C202, C203, C204, D201, D202, L201, Q201, R202, R203, R204, TR201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

Commit message: Found IC for ORing function. Added all LCSC refs. Found proper header stackup.
Signed-off-by: Jean Alinei <jean.alinei@owntech.org>
Parts:
- R202: LCSC (none) -> C15458
- TR201: LCSC (none) -> C37648313

Commit message: Added datasheets & updated components descriptions & values
Signed-off-by: Jean Alinei <jean.alinei@owntech.org>
Parts:
- D201, D202: value PMEG4010 -> PMEG4010ESBYL
Changed lines of the file:
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@@
 			)
 		)
-		(property "Description" "Unpolarized capacitor"
+		(property "Description" "10uF ±10% 50V Ceramic Capacitor X5R 0805"
 			(at 175.26 40.64 0)
 			(hide yes)
@@
 			)
 		)
-		(property "Value" "PMEG4010"
+		(property "Value" "PMEG4010ESBYL"
 			(at 156.718 51.054 0)
 			(show_name no)
@@
 			)
 		)
-		(property "Description" "Schottky diode, small symbol"
+		(property "Description" "Diode 40V 1A Surface Mount DSN1006-2"
 			(at 152.4 53.34 0)
 			(hide yes)
@@
 			)
 		)
-		(property "Description" "0.115A Id, 60V Vds, N-Channel MOSFET, SOT-23"
+		(property "Description" "N-Channel 60V 115mA 0.225W Surface Mount SOT-23"
 			(at 87.63 46.99 0)
 			(hide yes)
@@
 			)
 		)
-		(property "Value" "PMEG4010"
+		(property "Value" "PMEG4010ESBYL"
 			(at 146.812 33.02 0)
 			(show_name no)
@@
 			)
 		)
-		(property "Description" "Schottky diode, small symbol"
+		(property "Description" "Diode 40V 1A Surface Mount DSN1006-2"
 			(at 152.4 35.56 0)
 			(hide yes)
@@
 			)
 		)
-		(property "Description" "Isolated power transformer driver"
+		(property "Description" "ESOP-8 Power Management - Specialized RoHS"
 			(at 110.49 44.45 0)
 			(hide yes)
@@
 			)
 		)
-		(property "Description" "Unpolarized capacitor"
+		(property "Description" "100nF ±10% 50V Ceramic Capacitor X7R 0603"
 			(at 62.23 45.72 0)
 			(hide yes)
@@
 			)
 		)
-		(property "Description" "Resistor, small symbol"
+		(property "Description" "100kΩ ±5% 100mW 0603 Thick Film Resistor"
 			(at 90.17 36.83 0)
 			(hide yes)
@@
 			)
 		)
-		(property "Description" "Unpolarized capacitor"
+		(property "Description" "10uF ±10% 50V Ceramic Capacitor X5R 0805"
 			(at 34.29 45.72 0)
 			(hide yes)
@@
 			)
 		)
-		(property "Description" "Inductor"
+		(property "Description" "350mA 10uH ±20% 150mA 470mΩ Multilayer inductor 0805 Fixed Inductors RoHS"
 			(at 41.91 33.02 0)
 			(hide yes)
@@
 			)
 		)
-		(property "Description" "Unpolarized capacitor"
+		(property "Description" "10uF ±10% 50V Ceramic Capacitor X5R 0805"
 			(at 48.26 45.72 0)
 			(hide yes)
